File: KiCAD/5mm_X-Band_LGR_BOTTOM/X-Band_EPR_LGR_BOTTOM.kicad_pcb (KiCad board)
At the start: 2 copper layers, 31.8 x 31.8 mm, 6 parts

Commit message: Updated B12T Logo for PCB LGR BOTTOM
Parts:
- removed the LOGO at (91.1, 100.0)
- added LOGO: Val**, B12T_Open_PCB_LGR:b12t-logo-lowres, B.Cu at (90.0, 100.0)
Changed lines of the file:
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@@
     (add_net GND)
   )
-  (module aesthetics:b12t-logo-lowres (layer B.Cu)
-    (at 91.11 100 90)
-    (fp_text reference LOGO (at 0 -3.556 90) (layer B.SilkS) hide
+  (module B12T_Open_PCB_LGR:b12t-logo-lowres (layer B.Cu)
+    (at 90 100 90)
+    (fp_text reference LOGO (at 0 -3.556 270) (layer B.SilkS) hide
       (effects (font (size 1.524 1.524) (thickness 0.3)) (justify mirror))
     )
-    (fp_text value Val** (at 0 3.302 90) (layer B.SilkS) hide
+    (fp_text value Val** (at 0 3.302 270) (layer B.SilkS) hide
       (effects (font (size 1.27 1.27) (thickness 0.15)) (justify mirror))
     )
@@
       (effects (font (size 1 1) (thickness 0.15)))
     )
-    (fp_circle (center 0 0) (end 2.75 0) (layer F.CrtYd) (width 0.05))
     (fp_circle (center 0 0) (end 2.5 0) (layer Cmts.User) (width 0.15))
+    (fp_circle (center 0 0) (end 2.75 0) (layer F.CrtYd) (width 0.05))
     (fp_text user %R (at 0.3 0) (layer F.Fab)
       (effects (font (size 1 1) (thickness 0.15)))
@@
       (effects (font (size 1 1) (thickness 0.15)))
     )
-    (fp_circle (center 0 0) (end 2.5 0) (layer Cmts.User) (width 0.15))
     (fp_circle (center 0 0) (end 2.75 0) (layer F.CrtYd) (width 0.05))
+    (fp_circle (center 0 0) (end 2.5 0) (layer Cmts.User) (width 0.15))
     (fp_text user %R (at 0.3 0) (layer F.Fab)
       (effects (font (size 1 1) (thickness 0.15)))
@@
       (effects (font (size 1 1) (thickness 0.15)))
     )
-    (fp_circle (center 0 0) (end 2.75 0) (layer F.CrtYd) (width 0.05))
     (fp_circle (center 0 0) (end 2.5 0) (layer Cmts.User) (width 0.15))
+    (fp_circle (center 0 0) (end 2.75 0) (layer F.CrtYd) (width 0.05))
     (fp_text user %R (at 0.3 0) (layer F.Fab)
       (effects (font (size 1 1) (thickness 0.15)))
@@
       (effects (font (size 1 1) (thickness 0.15)))
     )
-    (fp_circle (center 0 0) (end 2.5 0) (layer Cmts.User) (width 0.15))
     (fp_circle (center 0 0) (end 2.75 0) (layer F.CrtYd) (width 0.05))
+    (fp_circle (center 0 0) (end 2.5 0) (layer Cmts.User) (width 0.15))
     (fp_text user %R (at 0.3 0) (layer F.Fab)
       (effects (font (size 1 1) (thickness 0.15)))
@@
       (effects (font (size 1 1) (thickness 0.15)))
     )
-    (fp_circle (center 0 0) (end 4.85 0) (layer F.CrtYd) (width 0.05))
     (fp_circle (center 0 0) (end 4.6 0) (layer Cmts.User) (width 0.15))
+    (fp_circle (center 0 0) (end 4.85 0) (layer F.CrtYd) (width 0.05))
     (fp_text user %R (at 0.3 0) (layer F.Fab)
       (effects (font (size 1 1) (thickness 0.15)))
