File: KiCAD/5mm_X-Band_LGR/X-Band_EPR_LGR.sch (KiCad schematic (older format))
At the start: 5 parts

Commit message: Updating footprint library reference for PCB LGR
Parts:
- H1: footprint B12T_Open:5.2mm_3L2G_X-Band -> B12T_Open_PCB_LGR:5.2mm_3L2G_X-Band
Changed lines of the file:
@@
 F 0 "H1" H 2100 1549 50  0000 L CNN
 F 1 "MountingHole_Pad" H 2100 1458 50  0000 L CNN
-F 2 "B12T_Open:5.2mm_3L2G_X-Band" H 2000 1500 50  0001 C CNN
+F 2 "B12T_Open_PCB_LGR:5.2mm_3L2G_X-Band" H 2000 1500 50  0001 C CNN
 F 3 "~" H 2000 1500 50  0001 C CNN
 	1    2000 1500
